File: Eagle/StandardTransducer-V0.2dQ/V0.2dQ.sch (EAGLE design)
At the start: 72 parts, among them CON1 SPI, IC2 TL072D, IC3 LP298XS, IC4 LORA-RA_01_SOIC, J1 87758-0216, Q1 FDN360P, Q2 FDN360P, Q3 FDN360P, Q5 BSP75, U1 RN2483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

Commit message: New version of 02.dQ
Parts:
- removed C6: 0.1uF, rcl:C-EUC0805
- removed L2: 10uH, rcl:L-EUL1812
- added Q4: FDN360P, transistor-power:FDN360P
- added R14: 1k, rcl:R-EU_R0805
- added R19: 220k, rcl:R-EU_R0805
Connections:
- removed net A3: U$4.PF4(ADC4/TCK)
- removed net DVCC: C6.1, L2.2, Q3.S, R10.1, R11.2, R12.2, R18.2, R8.1
- removed net N$1: F1.2, L1.1, L2.1
- new net AVCCOPA: IC2P.V+, Q4.D
- new net N$3: Q4.G, R14.1, R19.1
- new net VIN: C11.1, F1.2, IC3.VIN, J1-2.S, L1.1, R10.1, R11.2, R12.2, R8.1
- net ANGND: now also IC4.GND@1, IC4.GND@3, JP5.4
- net AVCC: now also Q4.S, R19.2; no longer IC2P.V+
- net D+3V3: now also Q3.S, R18.2, U$4.PF4(ADC4/TCK)
- net D10*: now also U$4.PC6(OC3A/!OC4A); no longer U$4.PB6(OC1B/OC4B/ADC13)
- net D6*: now also U$4.PB4(ADC11); no longer U$4.PD7(OC4D/ADC10/T0)
- net D7*: now also U$4.PD7(OC4D/ADC10/T0); no longer U$4.PE6(INT.6/AIN0)
- net D8*: now also U$4.PB5(OC1A/ADC12/!OC4B); no longer U$4.PB4(ADC11)
- net D9*: now also U$4.PB6(OC1B/OC4B/ADC13); no longer U$4.PB5(OC1A/ADC12/!OC4B)
- net GND: no longer C6.2, IC4.GND@1, IC4.GND@3, JP5.4
- net RA1/2483: now also U$4.PE6(INT.6/AIN0); no longer U$4.PC6(OC3A/!OC4A)
- net VCC: no longer C11.1, IC3.VIN, J1-2.S
- net VOPA: now also R14.2
Other:
- note added: "Se cambia por un LP5907 que entrega 250 mA."
- moved on the sheet: C4, F1, L1
